File: pcb/QCB_board.kicad_pcb (KiCad board)
At the start: 2 copper layers, 30.1 x 128 mm, 58 parts, among them IC1 ST3232BDR, J1 100616-2, J2 39-29-3086, J3 DIN41612_02x32_AC, J4 Conn_01x04_Socket, J5 Conn_01x04_Socket, J6 Conn_01x05_Socket, J8 Conn_01x03_Socket, U1 USBLC6-2SC6, U2 CH340E, U3 M24C02-WMN

Commit message: Sch complete, starting pcb
Parts:
- removed JP10, JP11, JP12: SolderJumper_3_Bridged12, Jumper:SolderJumper-3_P1.3mm_Bridged12_Pad1.0x1.5mm
- removed TP11: TestPoint, TestPoint:TestPoint_Pad_D1.0mm
- added C17: 10u, Capacitor_SMD:C_1206_3216Metric_Pad1.33x1.80mm_HandSolder, F.Cu at (-131.3, 67.3)
- added C18: 100n, Capacitor_SMD:C_0603_1608Metric_Pad1.08x0.95mm_HandSolder, F.Cu at (-132.1, 55.2)
- added C19: 100n, Capacitor_SMD:C_0603_1608Metric_Pad1.08x0.95mm_HandSolder, F.Cu at (-132.1, 57.7)
- added C20: 1u, Capacitor_SMD:C_0603_1608Metric_Pad1.08x0.95mm_HandSolder, F.Cu at (-127.8, 35.1)
- added C21: 10u, Capacitor_SMD:C_1206_3216Metric_Pad1.33x1.80mm_HandSolder, F.Cu at (-131.3, 70.7)
- added C22: 100n, Capacitor_SMD:C_0603_1608Metric_Pad1.08x0.95mm_HandSolder, F.Cu at (-127.8, 37.6)
- added C23: 100n, Capacitor_SMD:C_0603_1608Metric_Pad1.08x0.95mm_HandSolder, F.Cu at (-127.8, 40.1)
- added C24: 100n, Capacitor_SMD:C_0603_1608Metric_Pad1.08x0.95mm_HandSolder, F.Cu at (-127.8, 42.6)
- added C25: 100n, Capacitor_SMD:C_0603_1608Metric_Pad1.08x0.95mm_HandSolder, F.Cu at (-127.8, 45.1)
- added C26: 100n, Capacitor_SMD:C_0603_1608Metric_Pad1.08x0.95mm_HandSolder, F.Cu at (-127.8, 47.6)
- added C27: 100n, Capacitor_SMD:C_0603_1608Metric_Pad1.08x0.95mm_HandSolder, F.Cu at (-127.8, 50.1)
- added C28: 1u, Capacitor_SMD:C_0603_1608Metric_Pad1.08x0.95mm_HandSolder, F.Cu at (-127.8, 52.7)
- added C29: 10u, Capacitor_SMD:C_1206_3216Metric_Pad1.33x1.80mm_HandSolder, F.Cu at (-131.3, 74.0)
- added C30: 100n, Capacitor_SMD:C_0603_1608Metric_Pad1.08x0.95mm_HandSolder, F.Cu at (-127.8, 55.2)
- added C31: 100n, Capacitor_SMD:C_0603_1608Metric_Pad1.08x0.95mm_HandSolder, F.Cu at (-127.8, 57.7)
- added C32: 100n, Capacitor_SMD:C_0603_1608Metric_Pad1.08x0.95mm_HandSolder, F.Cu at (-123.4, 35.1)
- added C33: 100n, Capacitor_SMD:C_0603_1608Metric_Pad1.08x0.95mm_HandSolder, F.Cu at (-123.4, 37.6)
- added C34: 1n, Capacitor_SMD:C_0603_1608Metric_Pad1.08x0.95mm_HandSolder, F.Cu at (-123.4, 40.1)
- added C35: 100n, Capacitor_SMD:C_0603_1608Metric_Pad1.08x0.95mm_HandSolder, F.Cu at (-123.4, 42.6)
- added C36: 100n, Capacitor_SMD:C_0603_1608Metric_Pad1.08x0.95mm_HandSolder, F.Cu at (-123.4, 45.1)
- added C37: 6,8n, Capacitor_SMD:C_0603_1608Metric_Pad1.08x0.95mm_HandSolder, F.Cu at (-123.4, 47.6)
- added C38: 6,8n, Capacitor_SMD:C_0603_1608Metric_Pad1.08x0.95mm_HandSolder, F.Cu at (-123.4, 50.1)
- added C39: 10n, Capacitor_SMD:C_0603_1608Metric_Pad1.08x0.95mm_HandSolder, F.Cu at (-123.4, 52.7)
- added C40: 10n, Capacitor_SMD:C_0603_1608Metric_Pad1.08x0.95mm_HandSolder, F.Cu at (-123.4, 55.2)
- added C41: 18p, Capacitor_SMD:C_0402_1005Metric_Pad0.74x0.62mm_HandSolder, F.Cu at (-110.4, 59.9)
- added C42: 18p, Capacitor_SMD:C_0402_1005Metric_Pad0.74x0.62mm_HandSolder, F.Cu at (-110.4, 61.9)
- added C43: 1nF/2kV, Capacitor_SMD:C_1206_3216Metric_Pad1.33x1.80mm_HandSolder, F.Cu at (-131.3, 77.4)
- added C44: 100n, Capacitor_SMD:C_0603_1608Metric_Pad1.08x0.95mm_HandSolder, F.Cu at (-55.8, 35.1)
- added C45: 100n, Capacitor_SMD:C_0603_1608Metric_Pad1.08x0.95mm_HandSolder, F.Cu at (-55.8, 37.6)
- added C46: 10u, Capacitor_SMD:C_1206_3216Metric_Pad1.33x1.80mm_HandSolder, F.Cu at (-50.6, 48.6)
- added C47: 100n, Capacitor_SMD:C_0603_1608Metric_Pad1.08x0.95mm_HandSolder, F.Cu at (-55.8, 40.1)
- added C48: 100n, Capacitor_SMD:C_0603_1608Metric_Pad1.08x0.95mm_HandSolder, F.Cu at (-55.8, 42.6)
- added C49: 10u, Capacitor_SMD:C_1206_3216Metric_Pad1.33x1.80mm_HandSolder, F.Cu at (-50.6, 51.9)
- added C50: 100n, Capacitor_SMD:C_0603_1608Metric_Pad1.08x0.95mm_HandSolder, F.Cu at (-55.8, 45.1)
- added C51: 100n, Capacitor_SMD:C_0603_1608Metric_Pad1.08x0.95mm_HandSolder, F.Cu at (-55.8, 47.6)
- added C52: 10u, Capacitor_SMD:C_1206_3216Metric_Pad1.33x1.80mm_HandSolder, F.Cu at (-50.6, 55.3)
- added C53: 100n, Capacitor_SMD:C_0603_1608Metric_Pad1.08x0.95mm_HandSolder, F.Cu at (-55.8, 50.1)
- added C54: 100n, Capacitor_SMD:C_0603_1608Metric_Pad1.08x0.95mm_HandSolder, F.Cu at (-55.8, 52.7)
- added C55: 10u, Capacitor_SMD:C_1206_3216Metric_Pad1.33x1.80mm_HandSolder, F.Cu at (-50.6, 58.6)
- added C56: 100n, Capacitor_SMD:C_0603_1608Metric_Pad1.08x0.95mm_HandSolder, F.Cu at (90.1, 63.4)
- added C57: 100n, Capacitor_SMD:C_0805_2012Metric, F.Cu at (90.2, 113.8)
- added C58: 100n, Capacitor_SMD:C_0805_2012Metric, F.Cu at (90.2, 115.8)
- added C59: 10u, Capacitor_SMD:C_1206_3216Metric_Pad1.33x1.80mm_HandSolder, F.Cu at (86.7, 99.7)
- added C60: 100n, Capacitor_SMD:C_0603_1608Metric_Pad1.08x0.95mm_HandSolder, F.Cu at (86.8, 105.3)
- added C61: 100n, Capacitor_SMD:C_0805_2012Metric, F.Cu at (90.2, 117.8)
- added C62: 100n, Capacitor_SMD:C_0805_2012Metric, F.Cu at (90.2, 119.8)
- added C63: 100n, Capacitor_SMD:C_0603_1608Metric_Pad1.08x0.95mm_HandSolder, F.Cu at (-95.4, 94.4)
- added C64: 100n, Capacitor_SMD:C_0805_2012Metric, F.Cu at (-95.3, 82.6)
- added C65: 100n, Capacitor_SMD:C_0805_2012Metric, F.Cu at (-95.3, 85.7)
- added C66: 10u, Capacitor_SMD:C_1206_3216Metric_Pad1.33x1.80mm_HandSolder, F.Cu at (-94.5, 117.6)
- added C67: 100n, Capacitor_SMD:C_0603_1608Metric_Pad1.08x0.95mm_HandSolder, F.Cu at (-95.4, 96.9)
- added C68: 100n, Capacitor_SMD:C_0805_2012Metric, F.Cu at (-95.3, 88.7)
- added C69: 100n, Capacitor_SMD:C_0805_2012Metric, F.Cu at (-95.3, 91.7)
- added C70: 100n, Capacitor_SMD:C_0603_1608Metric_Pad1.08x0.95mm_HandSolder, F.Cu at (-48.1, 94.4)
- added C71: 100n, Capacitor_SMD:C_0805_2012Metric, F.Cu at (-48.1, 82.6)
- added C72: 100n, Capacitor_SMD:C_0805_2012Metric, F.Cu at (-48.1, 85.7)
- added C73: 10u, Capacitor_SMD:C_1206_3216Metric_Pad1.33x1.80mm_HandSolder, F.Cu at (-47.3, 117.6)
- added C74: 100n, Capacitor_SMD:C_0603_1608Metric_Pad1.08x0.95mm_HandSolder, F.Cu at (-48.1, 96.9)
- added C75: 100n, Capacitor_SMD:C_0805_2012Metric, F.Cu at (-48.1, 88.7)
- added C76: 100n, Capacitor_SMD:C_0805_2012Metric, F.Cu at (-48.1, 91.7)
- added C77: 100n, Capacitor_SMD:C_0603_1608Metric_Pad1.08x0.95mm_HandSolder, F.Cu at (-71.8, 94.4)
- added C78: 100n, Capacitor_SMD:C_0805_2012Metric, F.Cu at (-71.7, 82.6)
- added C79: 100n, Capacitor_SMD:C_0805_2012Metric, F.Cu at (-71.7, 85.7)
- added C80: 10u, Capacitor_SMD:C_1206_3216Metric_Pad1.33x1.80mm_HandSolder, F.Cu at (-70.9, 117.6)
- added C81: 100n, Capacitor_SMD:C_0603_1608Metric_Pad1.08x0.95mm_HandSolder, F.Cu at (-71.8, 96.9)
- added C82: 100n, Capacitor_SMD:C_0805_2012Metric, F.Cu at (-71.7, 88.7)
- added C83: 100n, Capacitor_SMD:C_0805_2012Metric, F.Cu at (-71.7, 91.7)
- added D11: SMF5.0CA, Diode_SMD:D_SMF, F.Cu at (-39.0, 55.2)
- added D12: UT8413A, Package_DFN_QFN:Diodes_UDFN-10_1.0x2.5mm_P0.5mm, F.Cu at (85.2, 114.9)
- added D13: UT8413A, Package_DFN_QFN:Diodes_UDFN-10_1.0x2.5mm_P0.5mm, F.Cu at (-95.8, 130.0)
- added D14: UT8413A, Package_DFN_QFN:Diodes_UDFN-10_1.0x2.5mm_P0.5mm, F.Cu at (-48.6, 130.0)
- added D15: UT8413A, Package_DFN_QFN:Diodes_UDFN-10_1.0x2.5mm_P0.5mm, F.Cu at (-72.2, 130.0)
- added D2: ~, LED_SMD:LED_0603_1608Metric_Pad1.05x0.95mm_HandSolder, F.Cu at (-23.7, 101.6)
- added D3: ~, LED_SMD:LED_0603_1608Metric_Pad1.05x0.95mm_HandSolder, F.Cu at (-106.0, 51.6)
- added D4: ~, LED_SMD:LED_0603_1608Metric_Pad1.05x0.95mm_HandSolder, F.Cu at (-106.0, 54.2)
- added D5: ~, LED_SMD:LED_0603_1608Metric_Pad1.05x0.95mm_HandSolder, F.Cu at (-106.0, 56.8)
- added D6: ~, LED_SMD:LED_0603_1608Metric_Pad1.05x0.95mm_HandSolder, F.Cu at (-106.0, 59.4)
- added D7: ~, LED_SMD:LED_0603_1608Metric_Pad1.05x0.95mm_HandSolder, F.Cu at (-106.0, 62.0)
- added D8: ~, LED_SMD:LED_0603_1608Metric_Pad1.05x0.95mm_HandSolder, F.Cu at (-106.0, 64.6)
- added D9: UT8413A, Package_DFN_QFN:Diodes_UDFN-10_1.0x2.5mm_P0.5mm, F.Cu at (-102.1, 75.8)
- added F1: Polyfuse, Fuse:Fuse_1206_3216Metric_Pad1.42x1.75mm_HandSolder, F.Cu at (-39.0, 48.5)
- added FB1: 100 @ 100MHz, Inductor_SMD:L_0603_1608Metric_Pad1.05x0.95mm_HandSolder, F.Cu at (-123.4, 57.7)
- added FB2: 100 @ 100MHz, Inductor_SMD:L_0603_1608Metric_Pad1.05x0.95mm_HandSolder, F.Cu at (-119.1, 35.1)
- added FB3: 100 @ 100MHz, Inductor_SMD:L_0603_1608Metric_Pad1.05x0.95mm_HandSolder, F.Cu at (-119.1, 37.6)
- added FB4: 100 @ 100MHz, Inductor_SMD:L_0603_1608Metric_Pad1.05x0.95mm_HandSolder, F.Cu at (-119.1, 40.1)
- added FB5: 100 @ 100MHz, Inductor_SMD:L_0603_1608Metric_Pad1.05x0.95mm_HandSolder, F.Cu at (-119.1, 42.6)
- added H5: MountingHole_Pad, MountingHole:MountingHole_2.7mm_M2.5_DIN965_Pad, F.Cu at (128.9, 27.8)
- added H6: MountingHole_Pad, MountingHole:MountingHole_2.7mm_M2.5_DIN965_Pad, F.Cu at (128.9, 150.3)
- added H7: MountingHole_Pad, MountingHole:MountingHole_2.7mm_M2.5_DIN965_Pad, F.Cu at (154.3, 27.8)
- added H8: MountingHole_Pad, MountingHole:MountingHole_2.7mm_M2.5_DIN965_Pad, F.Cu at (154.3, 150.3)
- added J10: DIN41612_02x32_AC, Connector_DIN:DIN41612_C_2x32_Female_Vertical_THT, F.Cu at (151.8, 49.7)
- added J7: DIN41612_02x32_AC, Connector_DIN:DIN41612_C_2x32_Female_Vertical_THT, F.Cu at (75.6, 49.7)
- added J9: DIN41612_02x32_AC, Connector_DIN:DIN41612_C_2x32_Female_Vertical_THT, F.Cu at (126.4, 49.7)
- added JP2: SolderJumper_3_Bridged12, Jumper:SolderJumper-3_P1.3mm_Bridged12_Pad1.0x1.5mm, F.Cu at (-125.5, 75.0)
- added JP3: SolderJumper_2_Open, Jumper:SolderJumper-2_P1.3mm_Open_RoundedPad1.0x1.5mm, F.Cu at (-114.2, 60.7)
- added JP4: SolderJumper_2_Bridged, Jumper:SolderJumper-2_P1.3mm_Bridged_RoundedPad1.0x1.5mm, F.Cu at (-114.2, 64.3)
- added JP5: SolderJumper_2_Open, Jumper:SolderJumper-2_P1.3mm_Open_RoundedPad1.0x1.5mm, F.Cu at (-114.2, 67.8)
- added JP6: SolderJumper_3_Bridged12, Jumper:SolderJumper-3_P1.3mm_Bridged12_Pad1.0x1.5mm, F.Cu at (91.2, 72.8)
- added JP7: SolderJumper_3_Bridged12, Jumper:SolderJumper-3_P1.3mm_Bridged12_Pad1.0x1.5mm, F.Cu at (-94.7, 125.8)
- added JP8: SolderJumper_3_Bridged12, Jumper:SolderJumper-3_P1.3mm_Bridged12_Pad1.0x1.5mm, F.Cu at (-47.5, 125.8)
- added L2: LQH32PN101MN0L, Inductor_SMD:L_1210_3225Metric, F.Cu at (-44.8, 53.2)
- added R12: 49R9, Resistor_SMD:R_0603_1608Metric_Pad0.98x0.95mm_HandSolder, F.Cu at (-119.1, 47.6)
- added R13: 49R9, Resistor_SMD:R_0603_1608Metric_Pad0.98x0.95mm_HandSolder, F.Cu at (-119.1, 50.1)
- added R14: 49R9, Resistor_SMD:R_0603_1608Metric_Pad0.98x0.95mm_HandSolder, F.Cu at (-119.1, 52.7)
- added R15: 49R9, Resistor_SMD:R_0603_1608Metric_Pad0.98x0.95mm_HandSolder, F.Cu at (-119.1, 55.2)
- added R16: 49R9, Resistor_SMD:R_0603_1608Metric_Pad0.98x0.95mm_HandSolder, F.Cu at (-119.1, 57.7)
- added R17: 2R2, Resistor_SMD:R_0603_1608Metric, F.Cu at (-101.8, 51.6)
- added R18: 2R2, Resistor_SMD:R_0603_1608Metric, F.Cu at (-101.8, 54.1)
- added R19: 2R2, Resistor_SMD:R_0603_1608Metric, F.Cu at (-101.8, 56.6)
- added R20: 2R2, Resistor_SMD:R_0603_1608Metric, F.Cu at (-101.8, 59.1)
- added R21: 330, Resistor_SMD:R_0603_1608Metric_Pad0.98x0.95mm_HandSolder, F.Cu at (-114.7, 35.1)
- added R22: 10k, Resistor_SMD:R_0603_1608Metric_Pad0.98x0.95mm_HandSolder, F.Cu at (-114.7, 37.6)
- added R23: 10k, Resistor_SMD:R_0603_1608Metric_Pad0.98x0.95mm_HandSolder, F.Cu at (-114.7, 40.1)
- added R24: 330, Resistor_SMD:R_0603_1608Metric_Pad0.98x0.95mm_HandSolder, F.Cu at (-114.7, 42.6)
- added R25: 330, Resistor_SMD:R_0603_1608Metric_Pad0.98x0.95mm_HandSolder, F.Cu at (-114.7, 45.1)
- added R26: 330, Resistor_SMD:R_0603_1608Metric_Pad0.98x0.95mm_HandSolder, F.Cu at (-114.7, 47.6)
- added R27: 330, Resistor_SMD:R_0603_1608Metric_Pad0.98x0.95mm_HandSolder, F.Cu at (-114.7, 50.1)
- added R28: 2R2, Resistor_SMD:R_0603_1608Metric, F.Cu at (-101.8, 61.6)
- added R29: 2R2, Resistor_SMD:R_0603_1608Metric, F.Cu at (-101.8, 64.1)
- added R30: 330, Resistor_SMD:R_0603_1608Metric_Pad0.98x0.95mm_HandSolder, F.Cu at (-114.7, 52.7)
- added R31: 2R2, Resistor_SMD:R_0603_1608Metric, F.Cu at (-97.8, 51.6)
- added R32: 2R2, Resistor_SMD:R_0603_1608Metric, F.Cu at (-97.8, 54.1)
- added R33: 6k19, Resistor_SMD:R_0603_1608Metric, F.Cu at (-97.8, 56.6)
- added R34: 10k, Resistor_SMD:R_0603_1608Metric_Pad0.98x0.95mm_HandSolder, F.Cu at (-114.7, 55.2)
- added R35: 10k, Resistor_SMD:R_0603_1608Metric_Pad0.98x0.95mm_HandSolder, F.Cu at (-114.7, 57.7)
- added R36: 10k, Resistor_SMD:R_0603_1608Metric_Pad0.98x0.95mm_HandSolder, F.Cu at (-110.4, 35.1)
- added R37: 2R2, Resistor_SMD:R_0603_1608Metric, F.Cu at (-97.8, 59.1)
- added R38: 2R2, Resistor_SMD:R_0603_1608Metric, F.Cu at (-97.8, 61.6)
- added R39: 2R2, Resistor_SMD:R_0603_1608Metric, F.Cu at (-97.8, 64.1)
- added R40: 2R2, Resistor_SMD:R_0603_1608Metric, F.Cu at (-93.8, 51.6)
- added R41: 49R9, Resistor_SMD:R_0603_1608Metric_Pad0.98x0.95mm_HandSolder, F.Cu at (-110.4, 37.6)
- added R42: 49R9, Resistor_SMD:R_0603_1608Metric_Pad0.98x0.95mm_HandSolder, F.Cu at (-110.4, 40.1)
- added R43: 10R, Resistor_SMD:R_0603_1608Metric_Pad0.98x0.95mm_HandSolder, F.Cu at (-110.4, 42.6)
- added R44: 1M, Resistor_SMD:R_0603_1608Metric, F.Cu at (-93.8, 54.1)
- added R45: 82R, Resistor_SMD:R_0603_1608Metric_Pad0.98x0.95mm_HandSolder, F.Cu at (-110.4, 45.1)
- added R46: 82R, Resistor_SMD:R_0603_1608Metric_Pad0.98x0.95mm_HandSolder, F.Cu at (-110.4, 47.6)
- added R47: 2R2, Resistor_SMD:R_0603_1608Metric, F.Cu at (-93.8, 56.6)
- added R48: 2R2, Resistor_SMD:R_0603_1608Metric, F.Cu at (-93.8, 59.1)
- added R49: 2R2, Resistor_SMD:R_0603_1608Metric, F.Cu at (-93.8, 61.6)
- added R50: 2R2, Resistor_SMD:R_0603_1608Metric, F.Cu at (-93.8, 64.1)
- added R51: 2R2, Resistor_SMD:R_0603_1608Metric, F.Cu at (-89.8, 51.6)
- added R52: 2R2, Resistor_SMD:R_0603_1608Metric, F.Cu at (-89.8, 54.1)
- added R53: 2R2, Resistor_SMD:R_0603_1608Metric, F.Cu at (-89.8, 56.6)
- added R54: 2R2, Resistor_SMD:R_0603_1608Metric, F.Cu at (-89.8, 59.1)
- added R55: 75R, Resistor_SMD:R_0603_1608Metric_Pad0.98x0.95mm_HandSolder, F.Cu at (-110.4, 50.1)
- added R56: 75R, Resistor_SMD:R_0603_1608Metric_Pad0.98x0.95mm_HandSolder, F.Cu at (-110.4, 52.7)
- added R57: 150R, Resistor_SMD:R_0603_1608Metric_Pad0.98x0.95mm_HandSolder, F.Cu at (-110.4, 55.2)
- added R58: 150R, Resistor_SMD:R_0603_1608Metric_Pad0.98x0.95mm_HandSolder, F.Cu at (-110.4, 57.7)
- added R59: 10k, Resistor_SMD:R_0603_1608Metric_Pad0.98x0.95mm_HandSolder, F.Cu at (86.8, 69.1)
- added R60: 10k, Resistor_SMD:R_0603_1608Metric_Pad0.98x0.95mm_HandSolder, F.Cu at (85.0, 68.0)
- added R61: 10k, Resistor_SMD:R_0603_1608Metric_Pad0.98x0.95mm_HandSolder, F.Cu at (-95.4, 99.5)
- added R62: 10k, Resistor_SMD:R_0603_1608Metric_Pad0.98x0.95mm_HandSolder, F.Cu at (-95.4, 102.0)
- added R63: 10k, Resistor_SMD:R_0603_1608Metric_Pad0.98x0.95mm_HandSolder, F.Cu at (-48.1, 99.5)
- added R64: 10k, Resistor_SMD:R_0603_1608Metric_Pad0.98x0.95mm_HandSolder, F.Cu at (-48.1, 102.0)
- added R65: 10k, Resistor_SMD:R_0603_1608Metric_Pad0.98x0.95mm_HandSolder, F.Cu at (-71.8, 99.5)
- added R66: 10k, Resistor_SMD:R_0603_1608Metric_Pad0.98x0.95mm_HandSolder, F.Cu at (-71.8, 102.0)
- added T1: H1102NL, SamacSys_Parts:SOIC127P940X597-16N, F.Cu at (-122.3, 66.1)
- added TP5: TestPoint, TestPoint:TestPoint_Pad_D1.0mm, F.Cu at (-96.0, 111.3)
- added TP6: TestPoint, TestPoint:TestPoint_Pad_D1.0mm, F.Cu at (-96.0, 114.4)
- added TP7: TestPoint, TestPoint:TestPoint_Pad_D1.0mm, F.Cu at (-48.8, 111.3)
- added TP8: TestPoint, TestPoint:TestPoint_Pad_D1.0mm, F.Cu at (-48.8, 114.4)
- added U10: M24C02-WMN, Package_SO:SOIC-8_3.9x4.9mm_P1.27mm, F.Cu at (-46.1, 106.6)
- added U11: USBLC6-2SC6, Package_TO_SOT_SMD:SOT-23-6_Handsoldering, F.Cu at (-47.4, 121.7)
- added U12: M24C02-WMN, Package_SO:SOIC-8_3.9x4.9mm_P1.27mm, F.Cu at (-69.7, 106.6)
- added U13: USBLC6-2SC6, Package_TO_SOT_SMD:SOT-23-6_Handsoldering, F.Cu at (-71.0, 121.7)
- added U4: USBLC6-2SC6, Package_TO_SOT_SMD:SOT-23-6_Handsoldering, F.Cu at (-113.4, 72.0)
- added U5: USBLC6-2SC6, Package_TO_SOT_SMD:SOT-23-6_Handsoldering, F.Cu at (-113.4, 76.8)
- added U6: M24C02-WMN, Package_SO:SOIC-8_3.9x4.9mm_P1.27mm, F.Cu at (90.5, 67.8)
- added U7: USBLC6-2SC6, Package_TO_SOT_SMD:SOT-23-6_Handsoldering, F.Cu at (86.7, 102.7)
- added U8: M24C02-WMN, Package_SO:SOIC-8_3.9x4.9mm_P1.27mm, F.Cu at (-93.3, 106.6)
- added U9: USBLC6-2SC6, Package_TO_SOT_SMD:SOT-23-6_Handsoldering, F.Cu at (-94.6, 121.7)
- added Y1: ABM8G-12.000MHZ-18, Crystal:Crystal_SMD_Abracon_ABM8G-4Pin_3.2x2.5mm, F.Cu at (-42.2, 93.1)
- added Y2: 3225-25M-SR, Crystal:Crystal_SMD_3225-4Pin_3.2x2.5mm, F.Cu at (-89.6, 74.2)
- C12: value 10u -> 100n; footprint Capacitor_SMD:C_1206_3216Metric_Pad1.33x1.80mm_HandSolder -> Capacitor_SMD:C_0603_1608Metric_Pad1.08x0.95mm_HandSolder
- C15: value 10u -> 1nF/2kV
- C16, C7: value 100n -> 1u
- C3, C5, C8: value 100n -> 10u; footprint Capacitor_SMD:C_0603_1608Metric_Pad1.08x0.95mm_HandSolder -> Capacitor_SMD:C_1206_3216Metric_Pad1.33x1.80mm_HandSolder
- C4: value 1nF/2kV -> 10u
- D1: value LED -> ~; moved to F.Cu
- IC1: value ST3232BDR -> IP175G; footprint SamacSys_Parts:SOIC127P600X175-16N -> SamacSys_Parts:QFN40P600X600X90-49N-D
- J1: value 100616-2 -> Conn_01x03_Socket; footprint SamacSys_Parts:1006162 -> Connector_JST:JST_PH_B3B-PH-K_1x03_P2.00mm_Vertical; moved to F.Cu
- J2: value 39-29-3086 -> Conn_01x04_Socket; footprint Connector_Molex:Molex_Mini-Fit_Jr_5566-08A_2x04_P4.20mm_Vertical -> Connector_JST:JST_PH_B4B-PH-K_1x04_P2.00mm_Vertical; moved to F.Cu
- J3: value DIN41612_02x32_AC -> 100616-2; footprint Connector_DIN:DIN41612_C_2x32_Female_Vertical_THT -> SamacSys_Parts:1006162
- J4: value Conn_01x04_Socket -> Conn_01x04; footprint Connector_JST:JST_PH_B4B-PH-K_1x04_P2.00mm_Vertical -> Connector_PinHeader_1.00mm:PinHeader_1x04_P1.00mm_Vertical; moved to F.Cu
- J5: value Conn_01x04_Socket -> Conn_01x02; footprint Connector_JST:JST_PH_B4B-PH-K_1x04_P2.00mm_Vertical -> Connector_PinHeader_1.00mm:PinHeader_1x02_P1.00mm_Vertical; moved to F.Cu
- J6: value Conn_01x05_Socket -> 39-29-3086; footprint Connector_JST:JST_PH_B5B-PH-K_1x05_P2.00mm_Vertical -> Connector_Molex:Molex_Mini-Fit_Jr_5566-08A_2x04_P4.20mm_Vertical; moved to F.Cu
- J8: value Conn_01x03_Socket -> DIN41612_02x32_AC; footprint Connector_JST:JST_PH_B3B-PH-K_1x03_P2.00mm_Vertical -> Connector_DIN:DIN41612_C_2x32_Female_Vertical_THT; moved to F.Cu
- R1: value 49R9 -> 47k
- R10: value 10k -> 330
- R11: value 10k -> 49R9
- R2, R3, R6: value 49R9 -> 100k
- R4, R5: value 49R9 -> 330
- R7, R8: value 22R -> 10k; footprint Resistor_SMD:R_0402_1005Metric_Pad0.72x0.64mm_HandSolder -> Resistor_SMD:R_0603_1608Metric_Pad0.98x0.95mm_HandSolder
- R9: value 2K -> 2k7; footprint Resistor_SMD:R_0805_2012Metric_Pad1.20x1.40mm_HandSolder -> Resistor_SMD:R_0603_1608Metric_Pad0.98x0.95mm_HandSolder; moved to F.Cu
- U1: value USBLC6-2SC6 -> FE1.1s; footprint Package_TO_SOT_SMD:SOT-23-6_Handsoldering -> Package_SO:SSOP-28_3.9x9.9mm_P0.635mm
- U2: value CH340E -> 24LC02; footprint Package_SO:MSOP-10_3x3mm_P0.5mm -> Package_SO:SOIC-8_3.9x4.9mm_P1.27mm
- U3: value M24C02-WMN -> 24LC02
- moved C7 290.0 mm to (-132.1, 35.1), turned to 0 degrees
- moved C9 285.9 mm to (-132.1, 37.6), turned to 0 degrees
- moved C10 285.4 mm to (-132.1, 40.1)
- moved C12 285.4 mm to (-132.1, 45.1)
- moved C11 285.3 mm to (-132.1, 42.6)
- moved C16 279.0 mm to (-132.1, 52.7), turned to 0 degrees
- moved C8 278.3 mm to (-131.3, 60.6)
- moved C14 277.1 mm to (-132.1, 50.1), turned to 0 degrees
- moved C15 274.9 mm to (-131.3, 64.0)
- moved C13 274.5 mm to (-132.1, 47.6), turned to 0 degrees
- moved R11 263.4 mm to (-119.1, 45.1), turned to 0 degrees
- moved J3 253.5 mm to (-118.0, 104.0), turned to 90 degrees
- moved IC1 249.2 mm to (-99.7, 69.5), turned to 0 degrees
- moved J5 248.8 mm to (-99.0, 75.2)
- moved J1 244.7 mm to (-82.0, 49.1), turned to 0 degrees
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Connections:
- C1 pad 1: Net-(C1-Pad1) -> Earth
- C1 pad 2: Earth -> GND
- C10 pad 1: +3.3V -> REG_OUT
- C11 pad 1: +3.3V -> VDD10
- C12 pad 1: +3.3V -> VDD10
- C13 pad 1: Net-(D10-K) -> DVDD
- C14 pad 1: Net-(D10-K) -> DVDD
- C15 pad 1: Net-(D10-K) -> Net-(C15-Pad1)
- C15 pad 2: GND -> Earth
- C16 pad 1: GND -> +3.3V
- C16 pad 2: +3.3V -> GND
- C2 pad 1: +3.3V -> /USB_Switch/VUSB
- C3 pad 1: Net-(IC1-C1-) -> /USB_Switch/VUSB
- C3 pad 2: Net-(IC1-C1+) -> GND
- C4 pad 1: Earth -> /USB_Switch/3V3USB
- C5 pad 1: Net-(IC1-C2+) -> Net-(U1-VD18)
- C5 pad 2: Net-(IC1-C2-) -> GND
- C6 pad 1: GND -> /USB_Switch/3V3USB
- C6 pad 2: Net-(IC1-V+) -> GND
- C7 pad 1: GND -> REG_OUT
- C7 pad 2: Net-(IC1-V-) -> GND
- C8 pad 1: GND -> REG_OUT
- C8 pad 2: Net-(J5-Pin_1) -> GND
- C9 pad 1: GND -> REG_OUT
- C9 pad 2: Net-(U2-V3) -> GND
- D1 pad 1: GND -> Net-(D1-K)
- F2 pad 1: Net-(D10-K) -> Net-(D11-A1)
- F2 pad 2: /+3,3V_CONN -> +5V
- IC1 pad 1: Net-(IC1-C1+) -> /ETH_Switch/1TX1_N
- IC1 pad 10: /TTL_CTS -> /ETH_Switch/2TX2_P
- IC1 pad 11: /TTL_USART+ -> /ETH_Switch/2TX2_N
- IC1 pad 12: /TTL_USART- -> REG_IN
- IC1 pad 13: /RS232_RX -> VDD10
- IC1 pad 14: /RS232_TX -> /ETH_Switch/3RX3_P
- IC1 pad 15: GND -> /ETH_Switch/3RX3_N
- IC1 pad 16: +3.3V -> /ETH_Switch/3TX3_P
- IC1 pad 2: Net-(IC1-V+) -> /ETH_Switch/1TX1_P
- IC1 pad 3: Net-(IC1-C1-) -> /ETH_Switch/1RX1_N
- IC1 pad 4: Net-(IC1-C2+) -> /ETH_Switch/1RX1_P
- IC1 pad 5: Net-(IC1-C2-) -> Net-(IC1-BGRES)
- IC1 pad 6: Net-(IC1-V-) -> GND
- IC1 pad 7: /RS232_RTS -> REG_IN
- IC1 pad 8: /RS232_CTS -> /ETH_Switch/2RX2_P
- IC1 pad 9: /TTL_RTS -> /ETH_Switch/2RX2_N
- J1 pad 1: /TX+ -> /CON1/RS485+
- J1 pad 2: /TX- -> /CON1/RS485-
- J1 pad 3: /RX+ -> GND
- J2 pad 1: /+12V_CONN -> /USB_Switch/VUSB
- J2 pad 2: /-12V_CONN -> /USB_Switch/D+
- J2 pad 3: /+5V_CONN -> /USB_Switch/D-
- J2 pad 4: /+3,3V_CONN -> GND
- J4 pad 1: /VUSB -> +3.3V
- J4 pad 2: /D+ -> /ETH_Switch/I2C_SDA
- J4 pad 3: /D- -> /ETH_Switch/I2C_SCL
- J5 pad 1: Net-(J5-Pin_1) -> Net-(IC1-RESETB)
- J5 pad 2: /DP -> GND
- J6 pad 1: GND -> /CON1/+12V
- J6 pad 2: /RS232_RTS -> /CON1/-12V
- J6 pad 3: /RS232_CTS -> +5V
- J6 pad 4: /RS232_RX -> +3.3V
- J6 pad 5: /RS232_TX -> /CON1/+5Vsb
- JP1 pad 1: GND -> /USB_Switch/3V3USB
- JP1 pad 3: +3.3V -> GND
- JP9 pad 1: /USB_USART- -> GND
- JP9 pad 2: /USART- -> Net-(JP9-C)
- JP9 pad 3: /TTL_USART- -> +3.3V
- R1 pad 1: /GRX- -> /USB_Switch/VUSB
- R1 pad 2: Net-(R1-Pad2) -> /USB_Switch/VUSB
- R10 pad 1: /SDA -> GND
- R10 pad 2: +3.3V -> Net-(D2-K)
- R11 pad 1: /SCL -> Net-(J3-Pad8)
- R11 pad 2: +3.3V -> Net-(R11-Pad2)
- R2 pad 1: /GRX+ -> /USB_Switch/VUSB
- R2 pad 2: Net-(R1-Pad2) -> GND
- R3 pad 1: /GTX+ -> /USB_Switch/3V3USB
- R3 pad 2: Net-(R3-Pad2) -> Net-(U1-~{XRSTJ})
- R4 pad 1: /GTX- -> Net-(U1-LED2)
- R4 pad 2: Net-(R3-Pad2) -> /USB_Switch/3V3USB
- R5 pad 1: Net-(R1-Pad2) -> Net-(D1-A)
- R5 pad 2: Net-(C1-Pad1) -> /USB_Switch/3V3USB
- R6 pad 1: Net-(R3-Pad2) -> /USB_Switch/3V3USB
- R6 pad 2: Net-(C1-Pad1) -> Net-(U1-BUSJ)
- R7 pad 1: Net-(R7-Pad1) -> Net-(D1-K)
- R7 pad 2: /UD+ -> /USB_Switch/3V3USB
- R8 pad 1: Net-(R8-Pad1) -> Net-(U1-TESTJ/EESDA)
- R8 pad 2: /UD- -> /USB_Switch/3V3USB
- R9 pad 1: Net-(D1-A) -> GND
- R9 pad 2: Net-(U2-TNOW) -> Net-(U1-REXT)
- TP1 pad 1: /SDA -> /USB_Switch/VUSB
- TP10 pad 1: /RS485- -> /CON4/SCL
- TP2 pad 1: /SCL -> GND
- TP3 pad 1: /VUSB -> /CON1/SDA
- TP4 pad 1: GND -> /CON1/SCL
- TP9 pad 1: /RS485+ -> /CON4/SDA
- U1 pad 1: /DP -> GND
- U1 pad 2: GND -> Net-(U1-XOUT)
- U1 pad 3: /DN -> Net-(U1-XIN)
- U1 pad 4: Net-(R8-Pad1) -> /CON4/D-
- U1 pad 5: Net-(J5-Pin_1) -> /CON4/D+
- U1 pad 6: Net-(R7-Pad1) -> /USB_Switch/VUSB
- U2 pad 1: /UD+ -> GND
- U2 pad 2: /UD- -> GND
- U2 pad 4: /USB_RTS -> GND
- U2 pad 5: /USB_CTS -> Net-(U1-TESTJ/EESDA)
- U2 pad 6: Net-(U2-TNOW) -> Net-(D1-K)
- U2 pad 7: Net-(J5-Pin_1) -> Net-(JP1-C)
- U2 pad 8: /USB_USART- -> /USB_Switch/3V3USB
- U3 pad 5: /SDA -> /ETH_Switch/I2C_SDA
- U3 pad 6: /SCL -> /ETH_Switch/I2C_SCL
- U3 pad 7: Net-(JP1-C) -> Net-(JP2-C)
Routing:
- net Earth: track 256.4 -> 0.00 mm
- net /+5VSB_CONN: track 40.7 -> 0.00 mm
- net /RS485-: track 27.7 -> 0.00 mm
- net /TTL_USART-: track 27.3 -> 0.00 mm, vias 2 -> 0
- net /RS485+: track 26.5 -> 0.00 mm
- net +3.3V: track 42.6 -> 17.2 mm, vias 2 -> 0
- net /TTL_USART+: track 24.4 -> 0.00 mm, vias 2 -> 0
- net /CTS: track 23.2 -> 0.00 mm, vias 2 -> 0
- net /RX+: track 23.0 -> 0.00 mm
- net /RX-: track 22.8 -> 0.00 mm
- net /TTL_CTS: track 21.7 -> 0.00 mm, vias 2 -> 0
- net Net-(J5-Pin_1): track 21.5 -> 0.00 mm, vias 2 -> 0
- net /GRX+: track 21.2 -> 0.00 mm
- net /GRX-: track 21.1 -> 0.00 mm
- net /RTS: track 20.5 -> 0.00 mm, vias 2 -> 0
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- added copper zone on B.Cu, net Earth
- added copper zone on F.Cu, net Earth
- removed copper zone on B.Cu, net GND
- removed copper zone on F.Cu, net GND
Other:
- board size 30.1 x 128 mm -> 101.6 x 128.7 mm
- copper layers 2 -> 4
- board text removed: "+12V"
- board text removed: "+3,3V"
- board text removed: "+5V"
- board text removed: "+5Vsb"
- board text removed: "-12V"
- board text removed: "A"
- board text removed: "ACT"
- board text removed: "B"
- board text removed: "CTS"
- board text removed: "D+"
- board text removed: "D-"
- board text removed: "ETHERNET"
- board text removed: "GND"
- board text removed: "GND x3"
- board text removed: "PWR"
- board text removed: "RS232"
- board text removed: "RS485"
- board text removed: "RTS"
- board text removed: "RX"
- board text removed: "TX"
- board text removed: "USB"
- board text removed: "USB/UART"
- board text removed: "Vbus"

Commit message: Routing
Parts:
- removed C50, C51, C53, C54: 100n, Capacitor_SMD:C_0603_1608Metric_Pad1.08x0.95mm_HandSolder
- removed C52, C55: 10u, Capacitor_SMD:C_1206_3216Metric_Pad1.33x1.80mm_HandSolder
- removed D11: SMF5.0CA, Diode_SMD:D_SMF
- removed D9: UT8413A, Package_DFN_QFN:Diodes_UDFN-10_1.0x2.5mm_P0.5mm
- removed F2: Polyfuse, Fuse:Fuse_1206_3216Metric_Pad1.42x1.75mm_HandSolder
- removed L2: LQH32PN101MN0L, Inductor_SMD:L_1210_3225Metric
- added U14: USBLC6-2SC6, Package_TO_SOT_SMD:SOT-23-6_Handsoldering, B.Cu at (90.5, 46.2)
- C2, C3, C35, C36, C37, C38, C4, C40, C43, C5, C6, D1, D12, D13, D14, D15, D2, FB5, IC1, J1, J2, J3, J6, JP1, R10, R2, R3, R4, R41, R42, R43, R5, R55, R56, R57, R58, R6, R7, R8, R9, T1, TP1, U1, U2, Y1: moved to B.Cu
- R1: value 47k -> 0R/47k; moved to B.Cu
- moved C15 290.7 mm to (149.8, 138.4)
- moved R12 272.3 mm to (138.8, 134.9), turned to -90 degrees
- moved R14 272.2 mm to (140.3, 134.9), turned to -90 degrees
- moved R16 271.1 mm to (140.0, 137.6), turned to 180 degrees
- moved R11 270.3 mm to (135.8, 134.9), turned to -90 degrees
- moved R13 270.1 mm to (137.3, 134.9), turned to -90 degrees
- moved R15 268.7 mm to (136.7, 137.6)
- moved R47 266.8 mm to (166.6, 114.6)
- moved R48 266.8 mm to (166.6, 117.1)
- moved R49 266.8 mm to (166.6, 119.6)
- moved R50 266.8 mm to (166.6, 122.1)
- moved C43 263.3 mm to (124.7, 139.2)
- moved J3 258.7 mm to (139.1, 132.1)
- moved C38 255.7 mm to (121.4, 124.1), turned to 90 degrees
- moved C35 254.2 mm to (118.4, 120.8), turned to -90 degrees
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Connections:
- net +5V renamed /CON1/+5V_PWR
- net /CON1/+12V renamed /CON1/+12V_PWR
- net /CON1/-12V renamed /CON1/-12V_PWR
- C2 pad 1: /USB_Switch/VUSB -> /CON1/VUSB
- C28 pad 1: unconnected-(C28-Pad1) -> DVCC
- C29 pad 1: unconnected-(C29-Pad1) -> DVCC
- C3 pad 1: /USB_Switch/VUSB -> /CON1/VUSB
- C57 pad 1: /CON1/TX+ -> /CON1/CON_TX+
- C58 pad 1: /CON1/TX- -> /CON1/CON_TX-
- C59 pad 1: /USB_Switch/VUSB -> /CON1/VUSB
- C60 pad 2: /USB_Switch/VUSB -> /CON1/VUSB
- C61 pad 1: /CON1/RX+ -> /CON1/CON_RX+
- C62 pad 1: /CON1/RX- -> /CON1/CON_RX-
- C64 pad 1: /CON2/TX+ -> /CON2/CON_TX+
- C65 pad 1: /CON2/TX- -> /CON2/CON_TX-
- C66 pad 1: /USB_Switch/VUSB -> /CON1/VUSB
- C67 pad 2: /USB_Switch/VUSB -> /CON1/VUSB
- C68 pad 1: /CON2/RX+ -> /CON2/CON_RX+
- C69 pad 1: /CON2/RX- -> /CON2/CON_RX-
- C71 pad 1: /CON3/TX+ -> /CON3/CON_TX+
- C72 pad 1: /CON3/TX- -> /CON3/CON_TX-
- C73 pad 1: /USB_Switch/VUSB -> /CON1/VUSB
- C74 pad 2: /USB_Switch/VUSB -> /CON1/VUSB
- C75 pad 1: /CON3/RX+ -> /CON3/CON_RX+
- C76 pad 1: /CON3/RX- -> /CON3/CON_RX-
- C78 pad 1: /CON4/TX+ -> /CON4/CON_TX+
- C79 pad 1: /CON4/TX- -> /CON4/CON_TX-
- C80 pad 1: /USB_Switch/VUSB -> /CON1/VUSB
- C81 pad 2: /USB_Switch/VUSB -> /CON1/VUSB
- C82 pad 1: /CON4/RX+ -> /CON4/CON_RX+
- C83 pad 1: /CON4/RX- -> /CON4/CON_RX-
- F1 pad 2: +3.3V -> /CON1/+3.3V_PWR
- J10 pad a27: /CON4/TX+ -> /CON4/CON_TX+
- J10 pad a28: /CON4/TX- -> /CON4/CON_TX-
- J10 pad a5: +3.3V -> /CON1/+3.3V_PWR
- J10 pad c21: /USB_Switch/VUSB -> /CON1/VUSB
- J10 pad c27: /CON4/RX+ -> /CON4/CON_RX+
- J10 pad c28: /CON4/RX- -> /CON4/CON_RX-
- J10 pad c5: +3.3V -> /CON1/+3.3V_PWR
- J2 pad 1: /USB_Switch/VUSB -> /CON1/VUSB
- J2 pad 2: /USB_Switch/D+ -> /USB_Switch/D_P
- J2 pad 3: /USB_Switch/D- -> /USB_Switch/D_N
- J6 pad 4: +3.3V -> /CON1/+3.3V_PWR
- J7 pad a27: /CON1/TX+ -> /CON1/CON_TX+
- J7 pad a28: /CON1/TX- -> /CON1/CON_TX-
- J7 pad a5: +3.3V -> /CON1/+3.3V_PWR
- J7 pad c21: /USB_Switch/VUSB -> /CON1/VUSB
- J7 pad c27: /CON1/RX+ -> /CON1/CON_RX+
- J7 pad c28: /CON1/RX- -> /CON1/CON_RX-
- J7 pad c5: +3.3V -> /CON1/+3.3V_PWR
- J8 pad a27: /CON2/TX+ -> /CON2/CON_TX+
- J8 pad a28: /CON2/TX- -> /CON2/CON_TX-
- J8 pad a5: +3.3V -> /CON1/+3.3V_PWR
- J8 pad c21: /USB_Switch/VUSB -> /CON1/VUSB
- J8 pad c27: /CON2/RX+ -> /CON2/CON_RX+
- J8 pad c28: /CON2/RX- -> /CON2/CON_RX-
- J8 pad c5: +3.3V -> /CON1/+3.3V_PWR
- J9 pad a27: /CON3/TX+ -> /CON3/CON_TX+
- J9 pad a28: /CON3/TX- -> /CON3/CON_TX-
- J9 pad a5: +3.3V -> /CON1/+3.3V_PWR
- J9 pad c21: /USB_Switch/VUSB -> /CON1/VUSB
- J9 pad c27: /CON3/RX+ -> /CON3/CON_RX+
- J9 pad c28: /CON3/RX- -> /CON3/CON_RX-
- J9 pad c5: +3.3V -> /CON1/+3.3V_PWR
- R1 pad 1: /USB_Switch/VUSB -> Net-(U1-VBUSM)
- R1 pad 2: /USB_Switch/VUSB -> /CON1/VUSB
- R2 pad 1: /USB_Switch/VUSB -> Net-(U1-VBUSM)
- TP1 pad 1: /USB_Switch/VUSB -> /CON1/VUSB
- U1 pad 18: /USB_Switch/VUSB -> Net-(U1-VBUSM)
- U1 pad 20: /USB_Switch/VUSB -> /CON1/VUSB
- U1 pad 6: /USB_Switch/VUSB -> /CON3/D-
- U11 pad 3: /USB_Switch/VUSB -> /CON3/D-
- U11 pad 5: /USB_Switch/VUSB -> /CON1/VUSB
- U13 pad 5: /USB_Switch/VUSB -> /CON1/VUSB
- U4 pad 1: /ETH_Switch/TX4_P -> /ETH_Switch/TD+
- U4 pad 3: /ETH_Switch/TX4_N -> /ETH_Switch/TD-
- U4 pad 4: /ETH_Switch/TD- -> /ETH_Switch/TX4_N
- U4 pad 6: /ETH_Switch/TD+ -> /ETH_Switch/TX4_P
- U5 pad 1: /ETH_Switch/RX4_P -> /ETH_Switch/RD+
- U5 pad 3: /ETH_Switch/RX4_N -> /ETH_Switch/RD-
- U5 pad 4: /ETH_Switch/RD- -> /ETH_Switch/RX4_N
- U5 pad 6: /ETH_Switch/RD+ -> /ETH_Switch/RX4_P
- U7 pad 5: /USB_Switch/VUSB -> /CON1/VUSB
- U9 pad 5: /USB_Switch/VUSB -> /CON1/VUSB
Routing:
- net Earth: track 0.00 -> 416.9 mm, vias 0 -> 791
- net /CON1/+5Vsb: track 0.00 -> 162.5 mm, vias 0 -> 8
- net /CON1/VUSB: track 0.00 -> 149.3 mm, vias 0 -> 1
- net GND: track 30.5 -> 142.8 mm, vias 1 -> 19
- net /CON1/RS485-: track 0.00 -> 96.0 mm
- net /CON1/RS485+: track 0.00 -> 91.6 mm
- net /CON1/+12V_PWR: track 0.00 -> 89.1 mm
- net /CON1/-12V_PWR: track 0.00 -> 88.4 mm
- net /CON1/+5V_PWR: track 0.00 -> 87.7 mm
- net /CON1/+3.3V_PWR: track 0.00 -> 87.0 mm
- net +3.3V: track 17.2 -> 71.4 mm
- net /USB_Switch/3V3USB: track 0.00 -> 44.1 mm
- net /CON2/D-: track 0.00 -> 36.0 mm, vias 0 -> 2
- net /ETH_Switch/TX+: track 0.00 -> 35.5 mm, vias 0 -> 1
- net /USB_Switch/D+: track 0.00 -> 35.3 mm
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- added copper zone on In1.Cu, net Earth
- added copper zone on In2.Cu, net Earth
- added copper zone on B.Cu, net GND
- added copper zone on F.Cu, net GND
- added copper zone on In1.Cu, net GND
- added copper zone on In2.Cu, net GND
