File: pcb/QCB_board.kicad_sch (KiCad schematic)
At the start: 10 parts, among them J1 Conn_01x03_Socket

Commit message: More routing
Changed lines of the file:
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@@
 	(wire
 		(pts
-			(xy 76.2 205.74) (xy 201.93 205.74)
+			(xy 76.2 208.28) (xy 262.89 208.28)
 		)
 		(stroke
@@
 	(wire
 		(pts
-			(xy 257.81 214.63) (xy 257.81 125.73)
-		)
-		(stroke
-			(width 0)
-			(type default)
-		)
-	)
-	(wire
-		(pts
 			(xy 132.08 92.71) (xy 137.16 92.71)
 		)
@@
 	(wire
 		(pts
+			(xy 201.93 123.19) (xy 201.93 217.17)
+		)
+		(stroke
+			(width 0)
+			(type default)
+		)
+	)
+	(wire
+		(pts
 			(xy 142.24 196.85) (xy 76.2 196.85)
 		)
@@
 	(wire
 		(pts
-			(xy 76.2 214.63) (xy 257.81 214.63)
-		)
-		(stroke
-			(width 0)
-			(type default)
-		)
-	)
-	(wire
-		(pts
 			(xy 287.02 71.12) (xy 257.81 71.12)
 		)
@@
 	(wire
 		(pts
+			(xy 76.2 214.63) (xy 199.39 214.63)
+		)
+		(stroke
+			(width 0)
+			(type default)
+		)
+	)
+	(wire
+		(pts
 			(xy 137.16 71.12) (xy 81.28 71.12)
 		)
@@
 	(wire
 		(pts
+			(xy 76.2 200.66) (xy 255.27 200.66)
+		)
+		(stroke
+			(width 0)
+			(type default)
+		)
+	)
+	(wire
+		(pts
+			(xy 260.35 205.74) (xy 260.35 123.19)
+		)
+		(stroke
+			(width 0)
+			(type default)
+		)
+	)
+	(wire
+		(pts
 			(xy 273.05 163.83) (xy 273.05 107.95)
 		)
@@
 	(wire
 		(pts
+			(xy 76.2 219.71) (xy 204.47 219.71)
+		)
+		(stroke
+			(width 0)
+			(type default)
+		)
+	)
+	(wire
+		(pts
 			(xy 246.38 274.32) (xy 242.57 274.32)
 		)
@@
 	(wire
 		(pts
-			(xy 76.2 208.28) (xy 204.47 208.28)
-		)
-		(stroke
-			(width 0)
-			(type default)
-		)
-	)
-	(wire
-		(pts
 			(xy 102.87 105.41) (xy 102.87 140.97)
 		)
@@
 	(wire
 		(pts
-			(xy 76.2 219.71) (xy 262.89 219.71)
-		)
-		(stroke
-			(width 0)
-			(type default)
-		)
-	)
-	(wire
-		(pts
 			(xy 76.2 105.41) (xy 102.87 105.41)
 		)
@@
 	(wire
 		(pts
-			(xy 255.27 212.09) (xy 255.27 128.27)
-		)
-		(stroke
-			(width 0)
-			(type default)
-		)
-	)
-	(wire
-		(pts
 			(xy 207.01 116.84) (xy 207.01 138.43)
 		)
@@
 	(wire
 		(pts
-			(xy 76.2 217.17) (xy 260.35 217.17)
-		)
-		(stroke
-			(width 0)
-			(type default)
-		)
-	)
-	(wire
-		(pts
 			(xy 257.81 71.12) (xy 199.39 71.12)
 		)
@@
 	(wire
 		(pts
-			(xy 196.85 200.66) (xy 196.85 128.27)
-		)
-		(stroke
-			(width 0)
-			(type default)
-		)
-	)
-	(wire
-		(pts
-			(xy 199.39 125.73) (xy 199.39 203.2)
-		)
-		(stroke
-			(width 0)
-			(type default)
-		)
-	)
-	(wire
-		(pts
 			(xy 262.89 120.65) (xy 252.73 120.65)
 		)
@@
 	(wire
 		(pts
+			(xy 76.2 205.74) (xy 260.35 205.74)
+		)
+		(stroke
+			(width 0)
+			(type default)
+		)
+	)
+	(wire
+		(pts
 			(xy 265.43 138.43) (xy 280.67 138.43)
 		)
@@
 	(wire
 		(pts
+			(xy 76.2 217.17) (xy 201.93 217.17)
+		)
+		(stroke
+			(width 0)
+			(type default)
+		)
+	)
+	(wire
+		(pts
 			(xy 257.81 125.73) (xy 252.73 125.73)
 		)
@@
 	(wire
 		(pts
+			(xy 76.2 212.09) (xy 196.85 212.09)
+		)
+		(stroke
+			(width 0)
+			(type default)
+		)
+	)
+	(wire
+		(pts
 			(xy 201.93 76.2) (xy 139.7 76.2)
 		)
@@
 	(wire
 		(pts
+			(xy 199.39 125.73) (xy 199.39 214.63)
+		)
+		(stroke
+			(width 0)
+			(type default)
+		)
+	)
+	(wire
+		(pts
 			(xy 198.12 90.17) (xy 198.12 68.58)
 		)
@@
 	(wire
 		(pts
-			(xy 262.89 219.71) (xy 262.89 120.65)
-		)
-		(stroke
-			(width 0)
-			(type default)
-		)
-	)
-	(wire
-		(pts
 			(xy 246.38 271.78) (xy 246.38 274.32)
 		)
@@
 	(wire
 		(pts
+			(xy 257.81 203.2) (xy 257.81 125.73)
+		)
+		(stroke
+			(width 0)
+			(type default)
+		)
+	)
+	(wire
+		(pts
 			(xy 231.14 274.32) (xy 238.76 274.32)
 		)
@@
 	(wire
 		(pts
+			(xy 262.89 208.28) (xy 262.89 120.65)
+		)
+		(stroke
+			(width 0)
+			(type default)
+		)
+	)
+	(wire
+		(pts
 			(xy 100.33 144.78) (xy 100.33 107.95)
 		)
@@
 	(wire
 		(pts
-			(xy 204.47 208.28) (xy 204.47 120.65)
-		)
-		(stroke
-			(width 0)
-			(type default)
-		)
-	)
-	(wire
-		(pts
 			(xy 95.25 135.89) (xy 147.32 135.89)
 		)
@@
 	(wire
 		(pts
-			(xy 76.2 200.66) (xy 196.85 200.66)
-		)
-		(stroke
-			(width 0)
-			(type default)
-		)
-	)
-	(wire
-		(pts
 			(xy 147.32 114.3) (xy 147.32 135.89)
 		)
@@
 	(wire
 		(pts
+			(xy 76.2 203.2) (xy 257.81 203.2)
+		)
+		(stroke
+			(width 0)
+			(type default)
+		)
+	)
+	(wire
+		(pts
 			(xy 100.33 107.95) (xy 76.2 107.95)
 		)
@@
 	(wire
 		(pts
-			(xy 201.93 205.74) (xy 201.93 123.19)
-		)
-		(stroke
-			(width 0)
-			(type default)
-		)
-	)
-	(wire
-		(pts
-			(xy 76.2 212.09) (xy 255.27 212.09)
-		)
-		(stroke
-			(width 0)
-			(type default)
-		)
-	)
-	(wire
-		(pts
 			(xy 134.62 189.23) (xy 134.62 128.27)
 		)
@@
 	(wire
 		(pts
+			(xy 204.47 120.65) (xy 204.47 219.71)
+		)
+		(stroke
+			(width 0)
+			(type default)
+		)
+	)
+	(wire
+		(pts
 			(xy 279.4 142.24) (xy 279.4 140.97)
 		)
@@
 	(wire
 		(pts
-			(xy 260.35 217.17) (xy 260.35 123.19)
-		)
-		(stroke
-			(width 0)
-			(type default)
-		)
-	)
-	(wire
-		(pts
 			(xy 86.36 185.42) (xy 86.36 120.65)
 		)
@@
 	(wire
 		(pts
-			(xy 199.39 203.2) (xy 76.2 203.2)
-		)
-		(stroke
-			(width 0)
-			(type default)
-		)
-	)
-	(wire
-		(pts
 			(xy 132.08 120.65) (xy 142.24 120.65)
 		)
@@
 		)
 		(stroke
+			(width 0)
+			(type default)
+		)
+	)
+	(wire
+		(pts
+			(xy 196.85 128.27) (xy 196.85 212.09)
+		)
+		(stroke
+			(width 0)
+			(type default)
+		)
+	)
+	(wire
+		(pts
+			(xy 255.27 200.66) (xy 255.27 128.27)
+		)
+		(stroke

Commit message: Add design review docs, expand README, sync PCB routing and production outputs
Routing progress on schematic/PCB, generated production outputs (gerbers,
BOM, PDFs), 3D model cache, and datasheet sync. Adds doc/ (design review
report + TODO) and README overview of architecture/status/repo layout.
Analysis tool output moved to .gitignore (regenerable, not source).
Parts:
- C1: footprint Capacitor_SMD:C_1206_3216Metric_Pad1.33x1.80mm_HandSolder -> Capacitor_SMD:C_1206_3216Metric
Connections:
- no-connect marks 0 -> 4
Changed lines of the file:
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@@
 		(color 0 0 0 0)
+	)
+	(no_connect
+		(at 76.2 101.6)
+	)
+	(no_connect
+		(at 132.08 101.6)
+	)
+	(no_connect
+		(at 194.31 101.6)
+	)
+	(no_connect
+		(at 252.73 101.6)
 	)
 	(wire
@@
 			)
 		)
-		(property "Footprint" "Capacitor_SMD:C_1206_3216Metric_Pad1.33x1.80mm_HandSolder"
+		(property "Footprint" "Capacitor_SMD:C_1206_3216Metric"
 			(at 204.47 267.0048 0)
 			(hide yes)

Commit message: Apply review checklist fixes, add fiducials, regenerate production outputs
- C41/C42 (Y2 load caps) now included in BOM
- Add USB hub crystal load caps C50/C51 (DNP), rework Y1 area placement
- 2 fiducials per side (hand assembly)
- Add IP175G, FE1.1s and UT8413A datasheets to doc/datasheet
- README: status updated (ready for prototype order), production links
- .gitignore: drop leftover SCA_board ibom.config.ini entry
- Regenerate BOM, PDFs, gerber zip, interactive BOM and 3D renders
Parts:
- added FID1, FID2, FID3, FID4: Fiducial, Fiducial:Fiducial_0.5mm_Mask1mm, symbol Mechanical:Fiducial
