File: pcb/QCB_board.kicad_sch (KiCad schematic)
At the start: 14 parts, among them J1 Conn_01x03_Socket

Commit message: Fix BOM data: LED part numbers (D1-D8), BOM field cleanup, BOM export settings
Parts:
- C1: Manufacturer_Part_Number (none) -> 1206B102K202
- J1: now not fitted; now left out of the parts list
Changed lines of the file:
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@@
 		(body_style 1)
 		(exclude_from_sim no)
-		(in_bom yes)
-		(on_board yes)
-		(in_pos_files yes)
-		(dnp no)
+		(in_bom no)
+		(on_board yes)
+		(in_pos_files yes)
+		(dnp yes)
 		(property "Reference" "J1"
 			(at 287.02 138.4299 0)
@@
 			(hide yes)
 			(show_name no)
+			(do_not_autoplace no)
+			(effects
+				(font
+					(size 1.27 1.27)
+				)
+			)
+		)
+		(property "Manufacturer_Part_Number" "1206B102K202"
+			(at 200.66 267.97 90)
+			(hide yes)
+			(show_name no)
