File: pcb/eth_switch.kicad_sch (KiCad schematic)
At the start: 109 parts, among them IC1 IP175G, J3 100616-2, J4 Conn_01x04, J5 Conn_01x02, T1 H1102NL, U3 24LC02, U4 USBLC6-2SC6, U5 USBLC6-2SC6, Y2 3225-25M-SR

Commit message: More routing
Parts:
- D3, D4, D5, D6, D7, D8: value ~ -> (none)

Commit message: Add design review docs, expand README, sync PCB routing and production outputs
Routing progress on schematic/PCB, generated production outputs (gerbers,
BOM, PDFs), 3D model cache, and datasheet sync. Adds doc/ (design review
report + TODO) and README overview of architecture/status/repo layout.
Analysis tool output moved to .gitignore (regenerable, not source).
Parts:
- removed C10, C31, C32: 100n, Capacitor_SMD:C_0603_1608Metric_Pad1.08x0.95mm_HandSolder, symbol Device:C
- C11, C12, C13, C14, C16, C18, C19, C20, C22, C23, C24, C25, C26, C27, C28, C30, C33, C34, C35, C36, C37, C38, C39, C40, C7, C9: footprint Capacitor_SMD:C_0603_1608Metric_Pad1.08x0.95mm_HandSolder -> Capacitor_SMD:C_0603_1608Metric
- C15, C17, C21, C29, C43, C8: footprint Capacitor_SMD:C_1206_3216Metric_Pad1.33x1.80mm_HandSolder -> Capacitor_SMD:C_1206_3216Metric
- C41, C42: footprint Capacitor_SMD:C_0402_1005Metric_Pad0.74x0.62mm_HandSolder -> Capacitor_SMD:C_0402_1005Metric
- D3, D4, D5, D6, D7, D8: footprint LED_SMD:LED_0603_1608Metric_Pad1.05x0.95mm_HandSolder -> LED_SMD:LED_0603_1608Metric
- R11, R12, R13, R14, R15, R16, R21, R22, R23, R24, R25, R26, R27, R30, R34, R35, R36, R41, R42, R43, R45, R46, R55, R56, R57, R58: footprint Resistor_SMD:R_0603_1608Metric_Pad0.98x0.95mm_HandSolder -> Resistor_SMD:R_0603_1608Metric
Connections:
- net REG_IN renamed VDD33
Other:
- moved on the sheet: C7, C8, C9, JP3, JP5

Commit message: Unify passive values/footprints, add via-in-pad DRC rule, regen outputs
Parts:
- C37, C38: value 6,8n -> 6.8n
- R11, R12, R13, R14, R15, R16, R41, R42: value 49R9 -> 49.9
- R17, R18, R19, R20, R28, R29, R31, R32, R37, R38, R39, R40, R47, R48, R49, R50, R51, R52, R53, R54: value 2R2 -> 2.2
- R33: value 6k19 -> 6.19k
- R43: value 10R -> 10
- R45, R46: value 82R -> 82
- R55, R56: value 75R -> 75
- R57, R58: value 150R -> 150
Changed lines of the file:
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@@
 			)
 		)
-		(property "Value" "2R2"
+		(property "Value" "2.2"
 			(at 273.05 203.454 90)
 			(show_name no)
@@
 			)
 		)
-		(property "Value" "2R2"
+		(property "Value" "2.2"
 			(at 285.75 203.454 90)
 			(show_name no)
@@
 			)
 		)
-		(property "Value" "2R2"
+		(property "Value" "2.2"
 			(at 275.59 203.454 90)
 			(show_name no)
@@
 			)
 		)
-		(property "Value" "2R2"
+		(property "Value" "2.2"
 			(at 283.21 82.296 90)
 			(show_name no)
@@
 			)
 		)
-		(property "Value" "2R2"
+		(property "Value" "2.2"
 			(at 288.29 203.454 90)
 			(show_name no)
@@
 			)
 		)
-		(property "Value" "150R"
+		(property "Value" "150"
 			(at 537.21 212.0899 0)
 			(show_name no)
@@
 			)
 		)
-		(property "Value" "2R2"
+		(property "Value" "2.2"
 			(at 235.966 152.4 90)
 			(show_name no)
@@
 			)
 		)
-		(property "Value" "49R9"
+		(property "Value" "49.9"
 			(at 485.14 48.2599 0)
 			(show_name no)
@@
 			)
 		)
-		(property "Value" "6k19"
+		(property "Value" "6.19k"
 			(at 246.126 144.78 90)
 			(show_name no)
@@
 			)
 		)
-		(property "Value" "49R9"
+		(property "Value" "49.9"
 			(at 474.98 48.2599 0)
 			(show_name no)
@@
 			)
 		)
-		(property "Value" "75R"
+		(property "Value" "75"
 			(at 521.97 212.0899 0)
 			(show_name no)
@@
 			)
 		)
-		(property "Value" "2R2"
+		(property "Value" "2.2"
 			(at 235.966 139.7 90)
 			(show_name no)
@@
 			)
 		)
-		(property "Value" "49R9"
+		(property "Value" "49.9"
 			(at 518.16 43.1799 0)
 			(show_name no)
@@
 			)
 		)
-		(property "Value" "2R2"
+		(property "Value" "2.2"
 			(at 278.13 82.296 90)
 			(show_name no)
@@
 			)
 		)
-		(property "Value" "49R9"
+		(property "Value" "49.9"
 			(at 478.79 179.0699 0)
 			(show_name no)
@@
 			)
 		)
-		(property "Value" "2R2"
+		(property "Value" "2.2"
 			(at 290.83 203.454 90)
 			(show_name no)
@@
 			)
 		)
-		(property "Value" "2R2"
+		(property "Value" "2.2"
 			(at 235.966 134.62 90)
 			(show_name no)
@@
 			)
 		)
-		(property "Value" "2R2"
+		(property "Value" "2.2"
 			(at 275.59 82.296 90)
 			(show_name no)
@@
 			)
 		)
-		(property "Value" "49R9"
+		(property "Value" "49.9"
 			(at 480.06 58.4199 0)
 			(show_name no)
@@
 			)
 		)
-		(property "Value" "2R2"
+		(property "Value" "2.2"
 			(at 235.966 160.02 90)
 			(show_name no)
@@
 			)
 		)
-		(property "Value" "2R2"
+		(property "Value" "2.2"
 			(at 293.37 203.454 90)
 			(show_name no)
@@
 			)
 		)
-		(property "Value" "82R"
+		(property "Value" "82"
 			(at 464.82 208.2799 0)
 			(show_name no)
@@
 			)
 		)
-		(property "Value" "49R9"
+		(property "Value" "49.9"
 			(at 528.32 43.1799 0)
 			(show_name no)
@@
 			)
 		)
-		(property "Value" "2R2"
+		(property "Value" "2.2"
 			(at 278.13 203.454 90)
 			(show_name no)
@@
 			)
 		)
-		(property "Value" "49R9"
+		(property "Value" "49.9"
 			(at 523.24 53.3399 0)
 			(show_name no)
@@
 			)
 		)
-		(property "Value" "2R2"
+		(property "Value" "2.2"
 			(at 235.966 154.94 90)
 			(show_name no)
@@
 			)
 		)
-		(property "Value" "150R"
+		(property "Value" "150"
 			(at 546.1 212.0899 0)
 			(show_name no)
@@
 			)
 		)
-		(property "Value" "10R"
+		(property "Value" "10"
 			(at 487.68 179.0699 0)
 			(show_name no)
@@
 			)
 		)
-		(property "Value" "49R9"
+		(property "Value" "49.9"
 			(at 469.9 179.0699 0)
 			(show_name no)
@@
 			)
 		)
-		(property "Value" "6,8n"
+		(property "Value" "6.8n"
 			(at 480.06 200.152 0)
 			(show_name no)
@@
 			)
 		)
-		(property "Value" "2R2"
+		(property "Value" "2.2"
 			(at 235.966 137.16 90)
 			(show_name no)
@@
 			)
 		)
-		(property "Value" "2R2"
+		(property "Value" "2.2"
 			(at 280.67 203.454 90)
 			(show_name no)
@@
 			)
 		)
-		(property "Value" "2R2"
+		(property "Value" "2.2"
 			(at 280.67 82.296 90)
 			(show_name no)
@@
 			)
 		)
-		(property "Value" "82R"
+		(property "Value" "82"
 			(at 472.44 208.2799 0)
 			(show_name no)
@@
 			)
 		)
-		(property "Value" "2R2"
+		(property "Value" "2.2"
 			(at 235.966 157.48 90)
 			(show_name no)
@@
 			)
 		)
-		(property "Value" "75R"
+		(property "Value" "75"
 			(at 529.59 212.0899 0)
 			(show_name no)
@@
 			)
 		)
-		(property "Value" "2R2"
+		(property "Value" "2.2"
 			(at 235.966 142.24 90)
 			(show_name no)
@@
 			)
 		)
-		(property "Value" "6,8n"
+		(property "Value" "6.8n"
 			(at 480.06 205.232 0)
 			(show_name no)

Commit message: Apply review checklist fixes, add fiducials, regenerate production outputs
- C41/C42 (Y2 load caps) now included in BOM
- Add USB hub crystal load caps C50/C51 (DNP), rework Y1 area placement
- 2 fiducials per side (hand assembly)
- Add IP175G, FE1.1s and UT8413A datasheets to doc/datasheet
- README: status updated (ready for prototype order), production links
- .gitignore: drop leftover SCA_board ibom.config.ini entry
- Regenerate BOM, PDFs, gerber zip, interactive BOM and 3D renders
Parts:
- C41, C42: now in the parts list
Changed lines of the file:
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@@
 		(body_style 1)
 		(exclude_from_sim no)
-		(in_bom no)
+		(in_bom yes)
 		(on_board yes)
 		(in_pos_files yes)
@@
 		(body_style 1)
 		(exclude_from_sim no)
-		(in_bom no)
-		(on_board yes)
-		(in_pos_files yes)
+		(in_bom yes)
+		(on_board yes)
+		(in_pos_files yes)
