File: pcb/eth_switch.kicad_sch (KiCad schematic)
At the start: 106 parts, among them IC1 IP175G, J3 100616-2, J4 Conn_01x04, J5 Conn_01x02, T1 H1102NL, U3 24LC02, U4 USBLC6-2SC6, U5 USBLC6-2SC6, Y2 3225-25M-SR

Commit message: Fix BOM data: LED part numbers (D1-D8), BOM field cleanup, BOM export settings
Parts:
- C11, C12, C13, C14, C18, C19, C22, C23, C24, C25, C26, C27, C30, C33, C9: Manufacturer_Part_Number (none) -> GRM188R71H104KA93D
- C15: Manufacturer_Part_Number (none) -> 1206B102K202
- C16, C20, C28, C7: Manufacturer_Part_Number (none) -> CL10B105KA8NNNC
- C17, C21, C29, C8: Manufacturer_Part_Number (none) -> CL31B106KBHNNNE
- D3, D4, D5, D6, D7, D8: value (none) -> Green; Manufacturer_Part_Number (none) -> N0G69S04
- J4, J5: now not fitted; now left out of the parts list
- JP2, JP3, JP4, JP5: now not fitted
- R11, R12, R13, R14, R15, R16: Manufacturer_Part_Number (none) -> CRCW060349R9FKTABC
