File: pcb/pwr.kicad_sch (KiCad schematic)
At the start: 11 parts, among them J6 39-29-3086

Commit message: More routing
Parts:
- added TP11: TestPoint, TestPoint:TestPoint_Pad_D1.0mm, symbol Connector:TestPoint
Connections:
- net +3.3V: now also TP11.1

Commit message: Add design review docs, expand README, sync PCB routing and production outputs
Routing progress on schematic/PCB, generated production outputs (gerbers,
BOM, PDFs), 3D model cache, and datasheet sync. Adds doc/ (design review
report + TODO) and README overview of architecture/status/repo layout.
Analysis tool output moved to .gitignore (regenerable, not source).
Parts:
- C44, C45, C47, C48: footprint Capacitor_SMD:C_0603_1608Metric_Pad1.08x0.95mm_HandSolder -> Capacitor_SMD:C_0603_1608Metric
- C46, C49: footprint Capacitor_SMD:C_1206_3216Metric_Pad1.33x1.80mm_HandSolder -> Capacitor_SMD:C_1206_3216Metric

Commit message: Fix BOM data: LED part numbers (D1-D8), BOM field cleanup, BOM export settings
Parts:
- C44, C45, C47, C48: Manufacturer_Part_Number (none) -> GRM188R71H104KA93D
- C46, C49: Manufacturer_Part_Number (none) -> CL31B106KBHNNNE
- D10: Manufacturer_Part_Number (none) -> ESD5Z3.3T1G
- F1: value Polyfuse -> 1A; Manufacturer_Part_Number (none) -> 0ZCJ0150F2C
- L1: Manufacturer_Part_Number (none) -> LQH32PN101MN0L
- TP11, TP2: now not fitted; now left out of the parts list
Changed lines of the file:
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@@
+			)
+		)
+		(property "Manufacturer_Part_Number" "GRM188R71H104KA93D "
+			(at 85.09 104.14 0)
+			(hide yes)
+			(show_name no)
+			(do_not_autoplace no)
+			(effects
+				(font
+					(size 1.27 1.27)
+				)
 			)
 		)
@@
 			)
 		)
+		(property "Manufacturer_Part_Number" "CL31B106KBHNNNE"
+			(at 107.95 104.14 0)
+			(hide yes)
+			(show_name no)
+			(do_not_autoplace no)
+			(effects
+				(font
+					(size 1.27 1.27)
+				)
+			)
+		)
 		(pin "1"
 		)
@@
 			)
 		)
+		(property "Manufacturer_Part_Number" "GRM188R71H104KA93D "
+			(at 119.38 104.14 0)
+			(hide yes)
+			(show_name no)
+			(do_not_autoplace no)
+			(effects
+				(font
+					(size 1.27 1.27)
+				)
+			)
+		)
 		(pin "1"
 		)
@@
 			)
 		)
+		(property "Manufacturer_Part_Number" "ESD5Z3.3T1G"
+			(at 153.67 104.14 90)
+			(hide yes)
+			(show_name no)
+			(do_not_autoplace no)
+			(effects
+				(font
+					(size 1.27 1.27)
+				)
+			)
+		)
 		(pin "1"
 		)
@@
 			)
 		)
+		(property "Manufacturer_Part_Number" "LQH32PN101MN0L"
+			(at 114.3 99.06 90)
+			(hide yes)
+			(show_name no)
+			(do_not_autoplace no)
+			(effects
+				(font
+					(size 1.27 1.27)
+				)
+			)
+		)
 		(pin "2"
 		)
@@
 			)
 		)
-		(property "Value" "Polyfuse"
+		(property "Value" "1A"
 			(at 163.83 95.25 90)
 			(show_name no)
@@
 		(property "Description" "Resettable fuse, polymeric positive temperature coefficient"
 			(at 163.83 99.06 0)
+			(hide yes)
+			(show_name no)
+			(do_not_autoplace no)
+			(effects
+				(font
+					(size 1.27 1.27)
+				)
+			)
+		)
+		(property "Manufacturer_Part_Number" "0ZCJ0150F2C"
+			(at 163.83 99.06 90)
 			(hide yes)
 			(show_name no)
@@
 			)
 		)
+		(property "Manufacturer_Part_Number" "GRM188R71H104KA93D "
+			(at 130.81 104.14 0)
+			(hide yes)
+			(show_name no)
+			(do_not_autoplace no)
+			(effects
+				(font
+					(size 1.27 1.27)
+				)
+			)
+		)
 		(pin "1"
 		)
@@
 		(body_style 1)
 		(exclude_from_sim no)
-		(in_bom yes)
-		(on_board yes)
-		(in_pos_files yes)
-		(dnp no)
+		(in_bom no)
+		(on_board yes)
+		(in_pos_files yes)
+		(dnp yes)
 		(fields_autoplaced yes)
 		(property "Reference" "TP11"
@@
 			)
 		)
+		(property "Manufacturer_Part_Number" "GRM188R71H104KA93D "
+			(at 96.52 104.14 0)
+			(hide yes)
+			(show_name no)
+			(do_not_autoplace no)
+			(effects
+				(font
+					(size 1.27 1.27)
+				)
+			)
+		)
 		(pin "1"
 		)
@@
 		(body_style 1)
 		(exclude_from_sim no)
-		(in_bom yes)
-		(on_board yes)
-		(in_pos_files yes)
-		(dnp no)
+		(in_bom no)
+		(on_board yes)
+		(in_pos_files yes)
+		(dnp yes)
 		(fields_autoplaced yes)
 		(property "Reference" "TP2"
@@
 			(at 142.24 104.14 0)
 			(hide yes)
+			(show_name no)
+			(do_not_autoplace no)
+			(effects
+				(font
+					(size 1.27 1.27)
+				)
+			)
+		)
+		(property "Manufacturer_Part_Number" "CL31B106KBHNNNE"
+			(at 142.24 104.14 0)
+			(hide yes)
