File: pcb/usb_switch.kicad_sch (KiCad schematic)
At the start: 26 parts, among them J2 Conn_01x04_Socket, U1 FE1.1s, U14 USBLC6-2SC6, U2 24LC02, Y1 ABM8G-12.000MHZ-18

Commit message: Fix BOM data: LED part numbers (D1-D8), BOM field cleanup, BOM export settings
Parts:
- C2: Manufacturer_Part_Number (none) -> GRM188R71H104KA93D
- C3, C4, C5: Manufacturer_Part_Number (none) -> CL31B106KBHNNNE
- D1, D2: value (none) -> Green; Manufacturer_Part_Number (none) -> N0G69S04
- J2, TP1: now not fitted; now left out of the parts list
- JP1: now not fitted
Changed lines of the file:
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@@
+			)
+		)
+		(property "Manufacturer_Part_Number" "CL31B106KBHNNNE"
+			(at 130.81 49.53 0)
+			(hide yes)
+			(show_name no)
+			(do_not_autoplace no)
+			(effects
+				(font
+					(size 1.27 1.27)
+				)
 			)
 		)
@@
 		(body_style 1)
 		(exclude_from_sim no)
-		(in_bom yes)
-		(on_board yes)
-		(in_pos_files yes)
-		(dnp no)
+		(in_bom no)
+		(on_board yes)
+		(in_pos_files yes)
+		(dnp yes)
 		(property "Reference" "J2"
 			(at 39.37 72.3899 0)
@@
 			)
 		)
-		(property "Value" ""
+		(property "Value" "Green"
 			(at 178.562 86.36 0)
 			(show_name no)
@@
 		(property "Sim.Pins" "1=K 2=A"
 			(at 181.61 90.17 0)
+			(hide yes)
+			(show_name no)
+			(do_not_autoplace no)
+			(effects
+				(font
+					(size 1.27 1.27)
+				)
+			)
+		)
+		(property "Manufacturer_Part_Number" "N0G69S04"
+			(at 181.61 90.17 90)
 			(hide yes)
 			(show_name no)
@@
 			)
 		)
+		(property "Manufacturer_Part_Number" "GRM188R71H104KA93D "
+			(at 119.38 49.53 0)
+			(hide yes)
+			(show_name no)
+			(do_not_autoplace no)
+			(effects
+				(font
+					(size 1.27 1.27)
+				)
+			)
+		)
 		(pin "1"
 		)
@@
 		(on_board yes)
 		(in_pos_files yes)
-		(dnp no)
+		(dnp yes)
 		(property "Reference" "JP1"
 			(at 198.1201 110.49 90)
@@
 		(body_style 1)
 		(exclude_from_sim no)
-		(in_bom yes)
-		(on_board yes)
-		(in_pos_files yes)
-		(dnp no)
+		(in_bom no)
+		(on_board yes)
+		(in_pos_files yes)
+		(dnp yes)
 		(fields_autoplaced yes)
 		(property "Reference" "TP1"
@@
 			)
 		)
+		(property "Manufacturer_Part_Number" "CL31B106KBHNNNE"
+			(at 153.67 49.53 0)
+			(hide yes)
+			(show_name no)
+			(do_not_autoplace no)
+			(effects
+				(font
+					(size 1.27 1.27)
+				)
+			)
+		)
 		(pin "1"
 		)
@@
 			)
 		)
-		(property "Value" ""
+		(property "Value" "Green"
 			(at 164.592 109.22 0)
 			(show_name no)
@@
 		(property "Sim.Pins" "1=K 2=A"
 			(at 167.64 113.03 0)
+			(hide yes)
+			(show_name no)
+			(do_not_autoplace no)
+			(effects
+				(font
+					(size 1.27 1.27)
+				)
+			)
+		)
+		(property "Manufacturer_Part_Number" "N0G69S04"
+			(at 167.64 113.03 90)
 			(hide yes)
 			(show_name no)
@@
 			(at 140.97 49.53 0)
 			(hide yes)
+			(show_name no)
+			(do_not_autoplace no)
+			(effects
+				(font
+					(size 1.27 1.27)
+				)
+			)
+		)
+		(property "Manufacturer_Part_Number" "CL31B106KBHNNNE"
+			(at 140.97 49.53 0)
+			(hide yes)
